Commit message: init

File: models/09.urdf.xacro (robot description, xacro)
@@ -4,4 +4,5 @@
      ixy iyy iyz
      ixz iyz izz -->
+       <xacro:include filename="$(find turtlebot3_description)/urdf/common_properties.xacro"/>
   <xacro:property name="base_xy" value="0.5" />
   <xacro:property name="b_base_z" value="0.3" />
@@ -15,13 +16,5 @@
   <xacro:property name="base_mass" value="10" />
   <xacro:property name="base_xy2" value="${base_xy*base_xy}" />
-  <material name="blue">
-    <color rgba="0 0 0.8 1"/>
-  </material>
-  <material name="black">
-    <color rgba="0 0 0 1"/>
-  </material>
-  <material name="white">
-    <color rgba="1 1 1 1"/>
-  </material>
+  <!--default inertia macro-->
   <xacro:macro name="default_inertial" params="mass">
     <inertial>
@@ -30,14 +23,9 @@
     </inertial>
   </xacro:macro>
-  <xacro:macro name="cuboid_inertial" params="mass height"> <!--solid cuboid macro-->
+  <!--solid cuboid inertia macro-->
+  <xacro:macro name="cuboid_inertial" params="mass height">
     <inertial>
       <mass value="${mass}" />
       <inertia ixx="${(1/12)*mass*(height*height+base_xy2)}" ixy="0.0" ixz="0.0" iyy="${(1/12)*mass*(base_xy2*2)}" iyz="0.0" izz="${(1/12)*mass*(base_xy2+height*height)}" />
-    </inertial>
-  </xacro:macro>
-  <xacro:macro name="sphere_inertial" params="mass height radius"> <!--solid sphere macro-->
-    <inertial>
-      <mass value="${mass}" />
-      <inertia ixx="${(2/5)*mass*radius*radius}" ixy="0.0" ixz="0.0" iyy="${(2/5)*mass*radius*radius}}" iyz="0.0" izz="${(2/5)*mass*radius*radius}" />
     </inertial>
   </xacro:macro>

File: models/10.urdf.xacro (robot description, xacro)
@@ -4,4 +4,5 @@
      ixy iyy iyz
      ixz iyz izz -->
+       <xacro:include filename="$(find turtlebot3_description)/urdf/common_properties.xacro"/>
   <xacro:property name="base_xy" value="0.5" />
   <xacro:property name="b_base_z" value="0.3" />
@@ -15,13 +16,5 @@
   <xacro:property name="base_mass" value="10" />
   <xacro:property name="base_xy2" value="${base_xy*base_xy}" />
-  <material name="blue">
-    <color rgba="0 0 0.8 1"/>
-  </material>
-  <material name="black">
-    <color rgba="0 0 0 1"/>
-  </material>
-  <material name="white">
-    <color rgba="1 1 1 1"/>
-  </material>
+  <!--default inertia macro-->
   <xacro:macro name="default_inertial" params="mass">
     <inertial>
@@ -30,14 +23,9 @@
     </inertial>
   </xacro:macro>
-  <xacro:macro name="cuboid_inertial" params="mass height"> <!--solid cuboid macro-->
+  <!--solid cuboid inertia macro-->
+  <xacro:macro name="cuboid_inertial" params="mass height">
     <inertial>
       <mass value="${mass}" />
       <inertia ixx="${(1/12)*mass*(height*height+base_xy2)}" ixy="0.0" ixz="0.0" iyy="${(1/12)*mass*(base_xy2*2)}" iyz="0.0" izz="${(1/12)*mass*(base_xy2+height*height)}" />
-    </inertial>
-  </xacro:macro>
-  <xacro:macro name="sphere_inertial" params="mass height radius"> <!--solid sphere macro-->
-    <inertial>
-      <mass value="${mass}" />
-      <inertia ixx="${(2/5)*mass*radius*radius}" ixy="0.0" ixz="0.0" iyy="${(2/5)*mass*radius*radius}}" iyz="0.0" izz="${(2/5)*mass*radius*radius}" />
     </inertial>
   </xacro:macro>
@@ -122,4 +110,5 @@
     </link>
     <joint name="${prefix}_wheel_joint" type="continuous">
+      <axis rpy="0 0 0" xyz="0 1 0"/>
       <parent link="base_link"/>
       <child link="${prefix}_wheel"/>
